File: bak_test.kicad_pcb (KiCad board)
At the start: 2 copper layers, 150 x 100 mm, 208 parts, among them J1 HSP2_MX-502584-0670, J2 HSP2_MX-502584-0670, J3 HSP2_MX-502584-0670, J4 HSP2_MX-502584-0670, J5 HSP2_MX-502584-0670, J6 HSP2_MX-502584-0670, J7 CONN_02X01, J8 CONN_02X01, J9 microSD, P1 Gniazdo akumulatora, P2 Gniazdo akumulatora, P3 Gniazdo programatora SWD, T1 IRLML6401, T10 BSS138, T11 BSS138, T12 BSS138, T13 BSS138, T14 FDV304P, T2 IRLML6401, T3 IRLML6401, T4 IRLML6401, T5 IRLML6401, T6 IRLML6401, T7 BSS138, T8 BSS138, T9 BSS138, U1 MCP1755T-3302E/DC, U10 TPS3823, U11 STM32L051R8, U12 DS3231SN, U13 MCP1755T-3302E/DC, U14 MCP1755T-3302E/DC, U15 MIC29302, U16 DHT22, U17 M590E, U18 S25FL1275ABMGI101, U19 ESP-07, U2 MCP1755T-3302E/DC, U20 SIMHOLDER, U3 MCP1755T-3302E/DC, U4 MCP1755T-3302E/DC, U5 MCP1755T-3302E/DC, U6 MCP1755T-3302E/DC, U7 74LVX373M, U8 74LVX373M, U9 MAX3485, Y1 32.768 kHz, Y2 8 MHz

Commit message: rysowanie PCB
Parts:
- C29: moved to F.Cu
- moved C26 74.1 mm to (35.1, 140.7)
- moved C22 56.7 mm to (92.7, 115.6)
- moved R39 56.7 mm to (96.5, 115.6)
- moved R29 56.7 mm to (92.7, 118.1)
- moved R37 56.7 mm to (96.5, 120.7)
- moved R38 56.7 mm to (96.5, 118.1)
- moved U9 56.7 mm to (91.4, 123.2)
- moved R12 28.1 mm to (138.4, 160.0), turned to 0 degrees
- moved R18 28.0 mm to (142.2, 160.0)
- moved Y2 27.8 mm to (110.5, 128.3)
- moved C13 27.8 mm to (111.8, 116.8)
- moved C14 27.8 mm to (127.0, 130.8)
- moved C17 27.8 mm to (108.0, 116.8)
- moved C18 27.8 mm to (123.2, 133.3)
- moved C21 27.8 mm to (119.4, 133.3)
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Connections:
- BT1 pad 2: GND -> ~
- C1 pad 2: GND -> ~
- C10 pad 2: GND -> ~
- C11 pad 2: GND -> ~
- C12 pad 2: GND -> ~
- C13 pad 2: GND -> ~
- C14 pad 2: GND -> ~
- C15 pad 1: +3.3V -> ~
- C15 pad 2: GND -> ~
- C16 pad 1: +3.3V -> ~
- C16 pad 2: GND -> ~
- C17 pad 2: GND -> ~
- C18 pad 2: GND -> ~
- C19 pad 2: GND -> ~
- C2 pad 2: GND -> ~
- C20 pad 2: GND -> ~
- C21 pad 1: +3.3VSTM -> ~
- C21 pad 2: GND -> ~
- C22 pad 1: +3.3V -> ~
- C22 pad 2: GND -> ~
- C23 pad 1: +3.3V -> ~
- C23 pad 2: GND -> ~
- C24 pad 1: +3.3VSTM -> ~
- C24 pad 2: GND -> ~
- C25 pad 2: GND -> ~
- C26 pad 1: +3.3VSTM -> ~
- C26 pad 2: GND -> ~
- C27 pad 1: +3.3VSTM -> ~
- C27 pad 2: GND -> ~
- C28 pad 2: GND -> ~
- C29 pad 2: GND -> ~
- C3 pad 2: GND -> ~
- C30 pad 1: +3.3V -> ~
- C30 pad 2: GND -> ~
- C31 pad 2: GND -> ~
- C32 pad 2: GND -> ~
- C33 pad 1: +3.3VSTM -> ~
- C33 pad 2: GND -> ~
- C34 pad 1: +3.3VSTM -> ~
- C34 pad 2: GND -> ~
- C35 pad 2: GND -> ~
- C36 pad 1: +3.3VSTM -> ~
- C36 pad 2: GND -> ~
- C37 pad 1: +3.3V -> ~
- C37 pad 2: GND -> ~
- C38 pad 2: GND -> ~
- C39 pad 1: +3.3VSTM -> ~
- C39 pad 2: GND -> ~
- C4 pad 2: GND -> ~
- C40 pad 1: +3.3V -> ~
- C40 pad 2: GND -> ~
- C41 pad 2: GND -> ~
- C42 pad 2: GND -> ~
- C43 pad 2: GND -> ~
- C44 pad 2: GND -> ~
- C45 pad 2: GND -> ~
- C46 pad 2: GND -> ~
- C47 pad 2: GND -> ~
- C48 pad 1: +3.3VSTM -> ~
- C48 pad 2: GND -> ~
- C49 pad 2: GND -> ~
- C5 pad 2: GND -> ~
- C50 pad 1: +3.3V -> ~
- C50 pad 2: GND -> ~
- C51 pad 2: GND -> ~
- C52 pad 1: +3.3V -> ~
- C52 pad 2: GND -> ~
- C53 pad 2: GND -> ~
- C54 pad 1: +3.3VSTM -> ~
- C54 pad 2: GND -> ~
- C6 pad 2: GND -> ~
- C7 pad 2: GND -> ~
- C8 pad 2: GND -> ~
- C9 pad 2: GND -> ~
- D4 pad 1: GND -> ~
- F11 pad 2: +3.3V -> ~
- F7 pad 2: Net-(D1-Pad1) -> Net-(D1-Pad3)
- F8 pad 2: Net-(D1-Pad3) -> Net-(D1-Pad1)
- J1 pad 6: GND -> ~
- J2 pad 6: GND -> ~
- J3 pad 6: GND -> ~
- J4 pad 6: GND -> ~
- J5 pad 6: GND -> ~
- J6 pad 6: GND -> ~
- J9 pad 10: GND -> ~
- J9 pad 11: GND -> ~
- J9 pad 12: GND -> ~
- J9 pad 4: +3.3VSTM -> ~
- J9 pad 6: GND -> ~
- J9 pad 9: GND -> ~
- P1 pad 3: GND -> ~
- P2 pad 3: GND -> ~
- P3 pad 2: GND -> ~
- P3 pad 4: +3.3V -> ~
- R19 pad 2: GND -> ~
- R20 pad 2: GND -> ~
- R21 pad 2: GND -> ~
- R22 pad 2: GND -> ~
- R23 pad 2: GND -> ~
- R24 pad 2: GND -> ~
- R27 pad 1: GND -> ~
- R28 pad 1: GND -> ~
- R30 pad 2: +3.3VSTM -> ~
- R31 pad 1: +3.3V -> ~
- R32 pad 1: +3.3V -> ~
- R33 pad 1: +3.3V -> ~
- R34 pad 2: +3.3VSTM -> ~
- R35 pad 1: GND -> ~
- R36 pad 1: +3.3V -> ~
- R37 pad 1: GND -> ~
- R40 pad 2: +3.3V -> ~
- R43 pad 2: +3.3V -> ~
- R44 pad 2: +3.3V -> ~
- R48 pad 1: +3.3VSTM -> ~
- R50 pad 1: GND -> ~
- R54 pad 1: +3.3V -> ~
- R58 pad 1: +3.3V -> ~
- R59 pad 1: +3.3V -> ~
- T10 pad 2: GND -> ~
- T11 pad 2: GND -> ~
- T12 pad 2: GND -> ~
- T13 pad 2: GND -> ~
- T14 pad 2: +3.3V -> ~
- T7 pad 2: GND -> ~
- T8 pad 2: GND -> ~
- T9 pad 2: GND -> ~
- TP16 pad 1: Net-(D1-Pad1) -> Net-(D1-Pad3)
- TP17 pad 1: Net-(D1-Pad3) -> Net-(D1-Pad1)
- TP23 pad 1: +3.3VSTM -> ~
- TP24 pad 1: +3.3V -> ~
- TP31 pad 1: GND -> ~
- U1 pad 3: GND -> ~
- U1 pad 6: GND -> ~
- U10 pad 2: GND -> ~
- U10 pad 5: +3.3V -> ~
- U11 pad 1: +3.3VSTM -> ~
- U11 pad 12: GND -> ~
- U11 pad 13: +3.3VSTM -> ~
- U11 pad 18: GND -> ~
- U11 pad 19: +3.3VSTM -> ~
- U11 pad 31: GND -> ~
- U11 pad 32: +3.3VSTM -> ~
- U11 pad 47: GND -> ~
- U11 pad 48: +3.3VSTM -> ~
- U11 pad 54: GND -> Net-(U11-Pad54)
- U11 pad 55: GND -> Net-(U11-Pad55)
- U11 pad 56: GND -> Net-(U11-Pad56)
- U11 pad 57: GND -> Net-(U11-Pad57)
- U11 pad 58: GND -> Net-(U11-Pad58)
- U11 pad 61: GND -> Net-(U11-Pad61)
- U11 pad 62: GND -> Net-(U11-Pad62)
- U11 pad 63: GND -> ~
- U11 pad 64: +3.3VSTM -> ~
- U12 pad 10: GND -> ~
- U12 pad 11: GND -> ~
- U12 pad 12: GND -> ~
- U12 pad 13: GND -> ~
- U12 pad 5: GND -> ~
- U12 pad 6: GND -> ~
- U12 pad 7: GND -> ~
- U12 pad 8: GND -> ~
- U12 pad 9: GND -> ~
- U13 pad 3: GND -> ~
- U13 pad 4: +3.3VSTM -> ~
- U13 pad 6: GND -> ~
- U14 pad 3: GND -> ~
- U14 pad 4: +3.3V -> ~
- U14 pad 6: GND -> ~
- U15 pad 3: GND -> ~
- U15 pad 6: GND -> ~
- U16 pad 3: GND -> ~
- U16 pad 4: GND -> ~
- U17 pad 1: GND -> ~
- U17 pad 15: GND -> ~
- U17 pad 20: GND -> ~
- U17 pad 4: GND -> ~
- U18 pad 4: GND -> ~
- U18 pad 8: +3.3VSTM -> ~
- U19 pad 8: +3.3V -> ~
- U19 pad 9: GND -> ~
- U2 pad 3: GND -> ~
- U2 pad 6: GND -> ~
- U20 pad 4: GND -> ~
- U3 pad 3: GND -> ~
- U3 pad 6: GND -> ~
- U4 pad 1: /33ON6 -> Net-(U4-Pad1)
- U4 pad 2: ~ -> Net-(C4-Pad1)
- U4 pad 3: GND -> ~
- U4 pad 4: Net-(C4-Pad1) -> ~
- U4 pad 5: Net-(U4-Pad5) -> /33ON6
- U4 pad 6: GND -> ~
- U5 pad 3: GND -> ~
- U5 pad 6: GND -> ~
- U6 pad 3: GND -> ~
- U6 pad 6: GND -> ~
- U7 pad 10: GND -> ~
- U7 pad 18: GND -> ~
- U7 pad 20: +3.3V -> ~
- U7 pad 3: GND -> ~
- U8 pad 10: GND -> ~
- U8 pad 18: GND -> ~
- U8 pad 20: +3.3V -> ~
- U8 pad 3: GND -> ~
- U9 pad 5: GND -> ~
- U9 pad 8: +3.3V -> ~
Routing:
- net GND: track 238.4 -> 0.00 mm, vias 8 -> 0
- net Net-(C45-Pad1): track 116.2 -> 0.00 mm, vias 3 -> 0
- net /GSM_STAB_EN: track 67.5 -> 0.00 mm
- net /BAT2_POM: track 7.92 -> 0.00 mm
- net Net-(D1-Pad3): track 19.6 -> 11.7 mm
- net ~: track 90.6 -> 97.5 mm, vias 2 -> 0
- net /BAT1_POM: track 6.61 -> 0.00 mm
- net Net-(P2-Pad2): track 6.46 -> 0.00 mm
- net Net-(P1-Pad2): track 6.40 -> 0.00 mm
- net Net-(R49-Pad1): track 6.16 -> 0.00 mm
- net Net-(D1-Pad1): track 12.9 -> 15.9 mm
- removed copper zone on B.Cu, net GND
