File: test.kicad_pcb (KiCad board)
At the start: 2 copper layers, 208 parts, among them J1 HSP2_MX-502584-0670, J2 HSP2_MX-502584-0670, J3 HSP2_MX-502584-0670, J4 HSP2_MX-502584-0670, J5 HSP2_MX-502584-0670, J6 HSP2_MX-502584-0670, J7 CONN_02X01, J8 CONN_02X01, J9 microSD, P1 Gniazdo akumulatora, P2 Gniazdo akumulatora, P3 Gniazdo programatora SWD, T1 IRLML6401, T10 BSS138, T11 BSS138, T12 BSS138, T13 BSS138, T14 FDV304P, T2 IRLML6401, T3 IRLML6401, T4 IRLML6401, T5 IRLML6401, T6 IRLML6401, T7 BSS138, T8 BSS138, T9 BSS138, U1 MCP1755T-3302E/DC, U10 TPS3823, U11 STM32L051R8, U12 DS3231SN, U13 MCP1755T-3302E/DC, U14 MCP1755T-3302E/DC, U15 MIC29302, U16 DHT22, U17 M590E, U18 S25FL1275ABMGI101, U19 ESP-07, U2 MCP1755T-3302E/DC, U20 SIMHOLDER, U3 MCP1755T-3302E/DC, U4 MCP1755T-3302E/DC, U5 MCP1755T-3302E/DC, U6 MCP1755T-3302E/DC, U7 74LVX373M, U8 74LVX373M, U9 MAX3485, Y1 32.768 kHz, Y2 8 MHz

Commit message: rysowanie PCB
Parts:
- C29, U17, U19, U20: moved to B.Cu
- moved J9 110.3 mm to (106.9, 84.6), turned to 180 degrees
- moved C48 104.8 mm to (103.9, 94.2)
- moved C35 86.7 mm to (17.5, 108.5), turned to 90 degrees
- moved C26 79.8 mm to (106.2, 119.9)
- moved C22 56.7 mm to (137.9, 149.9)
- moved R39 56.7 mm to (141.7, 149.9)
- moved R29 56.7 mm to (137.9, 152.4)
- moved R37 56.7 mm to (141.7, 154.9)
- moved R38 56.7 mm to (141.7, 152.4)
- moved U9 56.7 mm to (136.7, 157.5)
- moved Y1 50.5 mm to (89.7, 110.9)
- moved U12 40.1 mm to (119.6, 103.6)
- moved C29 38.7 mm to (50.6, 119.6), turned to 270 degrees
- moved R44 35.4 mm to (148.5, 88.2)
- moved BT1 35.4 mm to (142.8, 89.0)
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Connections:
- BT1 pad 2: ~ -> GND
- C1 pad 2: ~ -> GND
- C10 pad 2: ~ -> GND
- C11 pad 2: ~ -> GND
- C12 pad 2: ~ -> GND
- C13 pad 2: ~ -> GND
- C14 pad 2: ~ -> GND
- C15 pad 1: ~ -> +3.3V
- C15 pad 2: ~ -> GND
- C16 pad 1: ~ -> +3.3V
- C16 pad 2: ~ -> GND
- C17 pad 2: ~ -> GND
- C18 pad 2: ~ -> GND
- C19 pad 2: ~ -> GND
- C2 pad 2: ~ -> GND
- C20 pad 2: ~ -> GND
- C21 pad 1: ~ -> +3.3VSTM
- C21 pad 2: ~ -> GND
- C22 pad 1: ~ -> +3.3V
- C22 pad 2: ~ -> GND
- C23 pad 1: ~ -> +3.3V
- C23 pad 2: ~ -> GND
- C24 pad 1: ~ -> +3.3VSTM
- C24 pad 2: ~ -> GND
- C25 pad 2: ~ -> GND
- C26 pad 1: ~ -> +3.3VSTM
- C26 pad 2: ~ -> GND
- C27 pad 1: ~ -> +3.3VSTM
- C27 pad 2: ~ -> GND
- C28 pad 2: ~ -> GND
- C29 pad 2: ~ -> GND
- C3 pad 2: ~ -> GND
- C30 pad 1: ~ -> +3.3V
- C30 pad 2: ~ -> GND
- C31 pad 2: ~ -> GND
- C32 pad 2: ~ -> GND
- C33 pad 1: ~ -> +3.3VSTM
- C33 pad 2: ~ -> GND
- C34 pad 1: ~ -> +3.3VSTM
- C34 pad 2: ~ -> GND
- C35 pad 2: ~ -> GND
- C36 pad 1: ~ -> +3.3VSTM
- C36 pad 2: ~ -> GND
- C37 pad 1: ~ -> +3.3V
- C37 pad 2: ~ -> GND
- C38 pad 2: ~ -> GND
- C39 pad 1: ~ -> +3.3VSTM
- C39 pad 2: ~ -> GND
- C4 pad 2: ~ -> GND
- C40 pad 1: ~ -> +3.3V
- C40 pad 2: ~ -> GND
- C41 pad 2: ~ -> GND
- C42 pad 2: ~ -> GND
- C43 pad 2: ~ -> GND
- C44 pad 2: ~ -> GND
- C45 pad 2: ~ -> GND
- C46 pad 2: ~ -> GND
- C47 pad 2: ~ -> GND
- C48 pad 1: ~ -> +3.3VSTM
- C48 pad 2: ~ -> GND
- C49 pad 2: ~ -> GND
- C5 pad 2: ~ -> GND
- C50 pad 1: ~ -> +3.3V
- C50 pad 2: ~ -> GND
- C51 pad 2: ~ -> GND
- C52 pad 1: ~ -> +3.3V
- C52 pad 2: ~ -> GND
- C53 pad 2: ~ -> GND
- C54 pad 1: ~ -> +3.3VSTM
- C54 pad 2: ~ -> GND
- C6 pad 2: ~ -> GND
- C7 pad 2: ~ -> GND
- C8 pad 2: ~ -> GND
- C9 pad 2: ~ -> GND
- D4 pad 1: ~ -> GND
- F11 pad 2: ~ -> +3.3V
- F7 pad 2: Net-(D1-Pad3) -> Net-(D1-Pad1)
- F8 pad 2: Net-(D1-Pad1) -> Net-(D1-Pad3)
- J1 pad 6: ~ -> GND
- J2 pad 6: ~ -> GND
- J3 pad 6: ~ -> GND
- J4 pad 6: ~ -> GND
- J5 pad 6: ~ -> GND
- J6 pad 6: ~ -> GND
- J9 pad 10: ~ -> GND
- J9 pad 11: ~ -> GND
- J9 pad 12: ~ -> GND
- J9 pad 4: ~ -> +3.3VSTM
- J9 pad 6: ~ -> GND
- J9 pad 9: ~ -> GND
- P1 pad 3: ~ -> GND
- P2 pad 3: ~ -> GND
- P3 pad 2: ~ -> GND
- P3 pad 4: ~ -> +3.3V
- R19 pad 2: ~ -> GND
- R20 pad 2: ~ -> GND
- R21 pad 2: ~ -> GND
- R22 pad 2: ~ -> GND
- R23 pad 2: ~ -> GND
- R24 pad 2: ~ -> GND
- R27 pad 1: ~ -> GND
- R28 pad 1: ~ -> GND
- R30 pad 2: ~ -> +3.3VSTM
- R31 pad 1: ~ -> +3.3V
- R32 pad 1: ~ -> +3.3V
- R33 pad 1: ~ -> +3.3V
- R34 pad 2: ~ -> +3.3VSTM
- R35 pad 1: ~ -> GND
- R36 pad 1: ~ -> +3.3V
- R37 pad 1: ~ -> GND
- R40 pad 2: ~ -> +3.3V
- R43 pad 2: ~ -> +3.3V
- R44 pad 2: ~ -> +3.3V
- R48 pad 1: ~ -> +3.3VSTM
- R50 pad 1: ~ -> GND
- R54 pad 1: ~ -> +3.3V
- R58 pad 1: ~ -> +3.3V
- R59 pad 1: ~ -> +3.3V
- T10 pad 2: ~ -> GND
- T11 pad 2: ~ -> GND
- T12 pad 2: ~ -> GND
- T13 pad 2: ~ -> GND
- T14 pad 2: ~ -> +3.3V
- T7 pad 2: ~ -> GND
- T8 pad 2: ~ -> GND
- T9 pad 2: ~ -> GND
- TP16 pad 1: Net-(D1-Pad3) -> Net-(D1-Pad1)
- TP17 pad 1: Net-(D1-Pad1) -> Net-(D1-Pad3)
- TP23 pad 1: ~ -> +3.3VSTM
- TP24 pad 1: ~ -> +3.3V
- TP31 pad 1: ~ -> GND
- U1 pad 3: ~ -> GND
- U1 pad 6: ~ -> GND
- U10 pad 2: ~ -> GND
- U10 pad 5: ~ -> +3.3V
- U11 pad 1: ~ -> +3.3VSTM
- U11 pad 12: ~ -> GND
- U11 pad 13: ~ -> +3.3VSTM
- U11 pad 18: ~ -> GND
- U11 pad 19: ~ -> +3.3VSTM
- U11 pad 31: ~ -> GND
- U11 pad 32: ~ -> +3.3VSTM
- U11 pad 47: ~ -> GND
- U11 pad 48: ~ -> +3.3VSTM
- U11 pad 54: Net-(U11-Pad54) -> GND
- U11 pad 55: Net-(U11-Pad55) -> GND
- U11 pad 56: Net-(U11-Pad56) -> GND
- U11 pad 57: Net-(U11-Pad57) -> GND
- U11 pad 58: Net-(U11-Pad58) -> GND
- U11 pad 61: Net-(U11-Pad61) -> GND
- U11 pad 62: Net-(U11-Pad62) -> GND
- U11 pad 63: ~ -> GND
- U11 pad 64: ~ -> +3.3VSTM
- U12 pad 10: ~ -> GND
- U12 pad 11: ~ -> GND
- U12 pad 12: ~ -> GND
- U12 pad 13: ~ -> GND
- U12 pad 5: ~ -> GND
- U12 pad 6: ~ -> GND
- U12 pad 7: ~ -> GND
- U12 pad 8: ~ -> GND
- U12 pad 9: ~ -> GND
- U13 pad 3: ~ -> GND
- U13 pad 4: ~ -> +3.3VSTM
- U13 pad 6: ~ -> GND
- U14 pad 3: ~ -> GND
- U14 pad 4: ~ -> +3.3V
- U14 pad 6: ~ -> GND
- U15 pad 3: ~ -> GND
- U15 pad 6: ~ -> GND
- U16 pad 3: ~ -> GND
- U16 pad 4: ~ -> GND
- U17 pad 1: ~ -> GND
- U17 pad 15: ~ -> GND
- U17 pad 20: ~ -> GND
- U17 pad 4: ~ -> GND
- U18 pad 4: ~ -> GND
- U18 pad 8: ~ -> +3.3VSTM
- U19 pad 8: ~ -> +3.3V
- U19 pad 9: ~ -> GND
- U2 pad 3: ~ -> GND
- U2 pad 6: ~ -> GND
- U20 pad 4: ~ -> GND
- U3 pad 3: ~ -> GND
- U3 pad 6: ~ -> GND
- U4 pad 1: Net-(U4-Pad1) -> /33ON6
- U4 pad 2: Net-(C4-Pad1) -> ~
- U4 pad 3: ~ -> GND
- U4 pad 4: ~ -> Net-(C4-Pad1)
- U4 pad 5: /33ON6 -> Net-(U4-Pad5)
- U4 pad 6: ~ -> GND
- U5 pad 3: ~ -> GND
- U5 pad 6: ~ -> GND
- U6 pad 3: ~ -> GND
- U6 pad 6: ~ -> GND
- U7 pad 10: ~ -> GND
- U7 pad 18: ~ -> GND
- U7 pad 20: ~ -> +3.3V
- U7 pad 3: ~ -> GND
- U8 pad 10: ~ -> GND
- U8 pad 18: ~ -> GND
- U8 pad 20: ~ -> +3.3V
- U8 pad 3: ~ -> GND
- U9 pad 5: ~ -> GND
- U9 pad 8: ~ -> +3.3V
Routing:
- net GND: track 0.00 -> 238.4 mm, vias 0 -> 8
- net Net-(C45-Pad1): track 0.00 -> 116.2 mm, vias 0 -> 3
- net ~: track 0.00 -> 101.8 mm, vias 0 -> 2
- net /GSM_STAB_EN: track 0.00 -> 67.5 mm
- net Net-(C1-Pad1): track 0.00 -> 20.5 mm, vias 0 -> 2
- net Net-(D1-Pad3): track 0.00 -> 19.6 mm
- net Net-(D1-Pad1): track 0.00 -> 12.9 mm
- net /BAT2_POM: track 0.00 -> 7.92 mm
- net /BAT1_POM: track 0.00 -> 6.61 mm
- net Net-(P2-Pad2): track 0.00 -> 6.46 mm
- net Net-(P1-Pad2): track 0.00 -> 6.40 mm
- net Net-(R49-Pad1): track 0.00 -> 6.16 mm
- net Net-(F7-Pad1): track 0.00 -> 6.15 mm
- net Net-(F8-Pad1): track 0.00 -> 5.90 mm
- net Net-(F1-Pad1): track 0.00 -> 5.03 mm
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- added copper zone on B.Cu, net GND
Other:
- board outline added: 150 x 100 mm
- net class gruba added: clearance 0.4, trace_width 0.7, via_dia 1, via_drill 0.5

Commit message: rysowanie pcb
Parts:
- added REF** (x2): MX-502584-0670, footprints:MX-502584-0670, F.Cu at (0.00, 0.00)
- moved R37 144.1 mm to (-1.26, 172.7), turned to 90 degrees
- moved R38 144.0 mm to (-2.02, 161.3), turned to 270 degrees
- moved R39 141.4 mm to (0.78, 161.3), turned to 270 degrees
- moved C22 134.7 mm to (4.84, 170.9)
- moved U9 134.2 mm to (2.81, 167.4), turned to 270 degrees
- moved R29 130.9 mm to (7.89, 167.4), turned to 90 degrees
- moved C39 108.0 mm to (56.4, 110.5)
- moved C10 84.9 mm to (85.1, 150.9)
- moved C23 67.4 mm to (5.60, 159.3), turned to 180 degrees
- moved P3 55.7 mm to (115.1, 133.9)
- moved C21 23.4 mm to (116.6, 119.9)
- moved C24 16.1 mm to (113.0, 119.9)
- moved C14 15.2 mm to (87.9, 113.0), turned to 270 degrees
- moved C34 12.2 mm to (109.5, 119.9)
- moved C18 9.30 mm to (88.2, 121.4), turned to 90 degrees
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Connections:
- C10 pad 1: ~ -> VBAT
- C11 pad 1: ~ -> VBAT
- C12 pad 1: ~ -> VBAT
- C15 pad 1: +3.3V -> ~
- C16 pad 1: +3.3V -> ~
- C21 pad 1: +3.3VSTM -> ~
- C22 pad 1: +3.3V -> ~
- C23 pad 1: +3.3V -> ~
- C24 pad 1: +3.3VSTM -> ~
- C25 pad 1: ~ -> VBAT
- C26 pad 1: +3.3VSTM -> ~
- C27 pad 1: +3.3VSTM -> ~
- C28 pad 1: ~ -> VBAT
- C29 pad 1: ~ -> VBAT
- C30 pad 1: +3.3V -> ~
- C31 pad 1: ~ -> VBAT
- C32 pad 1: ~ -> VBAT
- C33 pad 1: +3.3VSTM -> ~
- C34 pad 1: +3.3VSTM -> ~
- C35 pad 1: ~ -> VBAT
- C36 pad 1: +3.3VSTM -> ~
- C37 pad 1: +3.3V -> ~
- C39 pad 1: +3.3VSTM -> ~
- C40 pad 1: +3.3V -> ~
- C48 pad 1: +3.3VSTM -> ~
- C50 pad 1: +3.3V -> ~
- C52 pad 1: +3.3V -> ~
- C54 pad 1: +3.3VSTM -> ~
- C7 pad 1: ~ -> VBAT
- C8 pad 1: ~ -> VBAT
- C9 pad 1: ~ -> VBAT
- D1 pad 4: ~ -> VBAT
- F10 pad 1: ~ -> VBAT
- F11 pad 2: +3.3V -> ~
- F9 pad 1: ~ -> VBAT
- J9 pad 4: +3.3VSTM -> ~
- P3 pad 4: +3.3V -> ~
- R10 pad 1: ~ -> VBAT
- R11 pad 1: ~ -> VBAT
- R12 pad 1: ~ -> VBAT
- R30 pad 2: +3.3VSTM -> ~
- R31 pad 1: +3.3V -> ~
- R32 pad 1: +3.3V -> ~
- R33 pad 1: +3.3V -> ~
- R34 pad 2: +3.3VSTM -> ~
- R36 pad 1: +3.3V -> ~
- R40 pad 2: +3.3V -> ~
- R43 pad 2: +3.3V -> ~
- R44 pad 2: +3.3V -> ~
- R48 pad 1: +3.3VSTM -> ~
- R54 pad 1: +3.3V -> ~
- R58 pad 1: +3.3V -> ~
- R59 pad 1: +3.3V -> ~
- R7 pad 1: ~ -> VBAT
- R8 pad 1: ~ -> VBAT
- R9 pad 1: ~ -> VBAT
- T1 pad 2: ~ -> VBAT
- T14 pad 2: +3.3V -> ~
- T2 pad 2: ~ -> VBAT
- T3 pad 2: ~ -> VBAT
- T4 pad 2: ~ -> VBAT
- T5 pad 2: ~ -> VBAT
- T6 pad 2: ~ -> VBAT
- TP23 pad 1: +3.3VSTM -> ~
- TP24 pad 1: +3.3V -> ~
- U1 pad 2: ~ -> VBAT
- U10 pad 5: +3.3V -> ~
- U11 pad 1: +3.3VSTM -> ~
- U11 pad 13: +3.3VSTM -> ~
- U11 pad 19: +3.3VSTM -> ~
- U11 pad 32: +3.3VSTM -> ~
- U11 pad 48: +3.3VSTM -> ~
- U11 pad 64: +3.3VSTM -> ~
- U13 pad 4: +3.3VSTM -> ~
- U14 pad 4: +3.3V -> ~
- U15 pad 2: ~ -> VBAT
- U18 pad 8: +3.3VSTM -> ~
- U19 pad 8: +3.3V -> ~
- U2 pad 2: ~ -> VBAT
- U3 pad 2: ~ -> VBAT
- U4 pad 2: ~ -> VBAT
- U5 pad 2: ~ -> VBAT
- U6 pad 2: ~ -> VBAT
- U7 pad 20: +3.3V -> ~
- U8 pad 20: +3.3V -> ~
- U9 pad 8: +3.3V -> ~
Routing:
- net GND: track 238.4 -> 540.6 mm, vias 8 -> 14
- net ~: track 101.8 -> 198.2 mm, vias 2 -> 6
- net VBAT: track 0.00 -> 85.3 mm, vias 0 -> 2
- net Net-(C2-Pad1): track 0.00 -> 21.6 mm, vias 0 -> 2
- net Net-(C1-Pad1): track 20.5 -> 41.0 mm, vias 2 -> 4
- net /VBON6: track 1.80 -> 12.6 mm
- net Net-(F1-Pad1): track 5.03 -> 10.1 mm
- net Net-(R13-Pad1): track 4.95 -> 9.91 mm
- net Net-(R17-Pad1): track 0.00 -> 4.95 mm
- net Net-(R16-Pad1): track 0.00 -> 4.95 mm
- net Net-(R15-Pad1): track 0.00 -> 4.95 mm
- net Net-(R14-Pad1): track 0.00 -> 4.95 mm
- net Net-(R18-Pad1): track 0.00 -> 4.95 mm
- net /BAT2_POM: track 7.92 -> 3.56 mm
- net Net-(F1-Pad2): track 3.66 -> 7.32 mm
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
Commit message: łączenie ścieżek pcb
Parts:
- removed the REF** at (0.00, 0.00)
- Y2: moved to B.Cu
- moved R38 113.4 mm to (93.5, 100.1), turned to 180 degrees
- moved R37 113.4 mm to (87.5, 102.1)
- moved R39 111.9 mm to (93.5, 98.5), turned to 180 degrees
- moved C23 44.6 mm to (46.0, 140.2), turned to 0 degrees
- moved C22 40.2 mm to (36.8, 146.6)
- moved R29 40.2 mm to (39.9, 143.0)
- moved U9 40.2 mm to (34.8, 143.0)
- moved C16 39.8 mm to (60.9, 135.2), turned to 270 degrees
- moved C27 38.0 mm to (88.9, 103.7), turned to 90 degrees
- moved C40 32.2 mm to (59.3, 100.7), turned to 270 degrees
- moved C24 30.2 mm to (85.8, 106.8), turned to 90 degrees
- moved R34 17.7 mm to (110.6, 123.8)
- moved U8 16.9 mm to (83.7, 139.1), turned to 90 degrees
- moved C26 16.3 mm to (89.9, 119.9), turned to 270 degrees
- moved R35 16.1 mm to (107.9, 123.8)
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Connections:
- C31 pad 1: VBAT -> Net-(C31-Pad1)
- C32 pad 1: VBAT -> Net-(C32-Pad1)
- F10 pad 2: Net-(F10-Pad2) -> Net-(C32-Pad1)
- F9 pad 2: Net-(F9-Pad2) -> Net-(C31-Pad1)
- R13 pad 2: /VBON6 -> /VBON1
- R14 pad 2: /VBON6 -> /VBON2
- R15 pad 2: /VBON6 -> /VBON3
- R16 pad 2: /VBON6 -> /VBON4
- R17 pad 2: /VBON6 -> /VBON5
- R19 pad 1: /VBON6 -> /VBON1
- R20 pad 1: /VBON6 -> /VBON2
- R21 pad 1: /VBON6 -> /VBON3
- R22 pad 1: /VBON6 -> /VBON4
- R23 pad 1: /VBON6 -> /VBON5
- TP10 pad 1: /VBON6 -> /VBON4
- TP11 pad 1: /VBON6 -> /VBON5
- TP19 pad 1: Net-(F10-Pad2) -> Net-(C32-Pad1)
- TP20 pad 1: Net-(F9-Pad2) -> Net-(C31-Pad1)
- TP7 pad 1: /VBON6 -> /VBON1
- TP8 pad 1: /VBON6 -> /VBON2
- TP9 pad 1: /VBON6 -> /VBON3
- U1 pad 1: /33ON6 -> /33ON1
- U13 pad 1: Net-(F10-Pad2) -> Net-(C32-Pad1)
- U13 pad 2: Net-(F10-Pad2) -> Net-(C32-Pad1)
- U14 pad 2: Net-(F9-Pad2) -> Net-(C31-Pad1)
- U2 pad 1: /33ON6 -> /33ON2
- U3 pad 1: /33ON6 -> /33ON3
- U4 pad 1: /33ON6 -> /33ON4
- U5 pad 1: /33ON6 -> /33ON5
Routing:
- net GND: track 540.6 -> 759.1 mm, vias 14 -> 16
- net ~: track 198.2 -> 316.9 mm, vias 6 -> 11
- net /485_RDE: track 0.00 -> 88.5 mm, vias 0 -> 2
- net /485_DI: track 0.00 -> 84.6 mm, vias 0 -> 2
- net /485_RO: track 0.00 -> 80.3 mm, vias 0 -> 2
- net /VON1: track 0.00 -> 66.8 mm, vias 0 -> 4
- net /33ON6: track 0.00 -> 66.4 mm, vias 0 -> 6
- net /VON3: track 0.00 -> 66.1 mm, vias 0 -> 4
- net /VON2: track 0.00 -> 66.0 mm, vias 0 -> 4
- net /33LOE: track 0.00 -> 53.7 mm, vias 0 -> 2
- net /VBON1: track 0.00 -> 51.3 mm
- net /VON6: track 0.00 -> 47.2 mm
- net /33ON1: track 0.00 -> 45.9 mm, vias 0 -> 2
- net /33ON5: track 0.00 -> 45.0 mm, vias 0 -> 4
- net /VON5: track 0.00 -> 43.7 mm, vias 0 -> 4
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Other:
- outline, holes or cut-outs redrawn
- net class Default: via_dia 0.6 -> 0.4; via_drill 0.4 -> 0.2
- rule via_min_drill: 0.3 -> 0.2

Commit message: rutowanie pcb
Parts:
- removed R51: 1k, Resistors_SMD:R_0603
- removed REF**: MX-502584-0670, footprints:MX-502584-0670
- removed TP1, TP2, TP3, TP4, TP5, TP6: TEST, Measurement_Points:Measurement_Point_Round-SMD-Pad_Big
- BT1, F11, U16: moved to B.Cu
- U20: moved to F.Cu
- moved TP10 222.3 mm to (69.5, 181.9)
- moved TP11 222.3 mm to (112.4, 182.3)
- moved TP13 222.3 mm to (54.6, 189.9)
- moved TP16 222.3 mm to (109.3, 189.5)
- moved TP18 222.3 mm to (58.4, 189.9)
- moved TP22 222.3 mm to (69.3, 188.7)
- moved TP23 222.3 mm to (55.4, 184.1)
- moved TP24 222.3 mm to (50.8, 189.9)
- moved TP26 222.3 mm to (98.9, 182.4)
- moved TP27 222.3 mm to (113.4, 189.5)
- moved TP28 222.3 mm to (73.4, 188.7)
- moved TP7 222.3 mm to (101.4, 189.5)
- moved TP8 222.3 mm to (105.3, 189.5)
- moved TP9 222.3 mm to (94.8, 182.4)
- moved TP12 222.3 mm to (83.5, 190.2)
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Connections:
- C15 pad 1: ~ -> +3.3V
- C16 pad 1: ~ -> +3.3V
- C21 pad 1: ~ -> +3.3VSTM
- C22 pad 1: ~ -> +3.3V
- C23 pad 1: ~ -> +3.3V
- C24 pad 1: ~ -> +3.3VSTM
- C26 pad 1: ~ -> +3.3VSTM
- C27 pad 1: ~ -> +3.3VSTM
- C30 pad 1: ~ -> +3.3VSTM
- C33 pad 1: ~ -> +3.3VSTM
- C34 pad 1: ~ -> +3.3VSTM
- C36 pad 1: ~ -> +3.3VSTM
- C37 pad 1: ~ -> +3.3V
- C39 pad 1: ~ -> +3.3VSTM
- C40 pad 1: ~ -> +3.3V
- C47 pad 1: Net-(C47-Pad1) -> +3.3V
- C48 pad 1: ~ -> +3.3VSTM
- C49 pad 1: Net-(C47-Pad1) -> Net-(C49-Pad1)
- C50 pad 1: ~ -> +3.3V
- C52 pad 1: ~ -> +3.3V
- C54 pad 1: ~ -> +3.3VSTM
- F11 pad 2: ~ -> +3.3V
- J9 pad 4: ~ -> +3.3VSTM
- P3 pad 4: ~ -> +3.3V
- R30 pad 2: ~ -> +3.3VSTM
- R31 pad 1: ~ -> +3.3V
- R32 pad 1: ~ -> +3.3V
- R33 pad 1: ~ -> +3.3V
- R34 pad 2: ~ -> +3.3VSTM
- R36 pad 1: ~ -> +3.3V
- R40 pad 2: ~ -> Net-(C43-Pad1)
- R43 pad 2: ~ -> +3.3V
- R44 pad 2: ~ -> Net-(C43-Pad1)
- R48 pad 1: ~ -> +3.3VSTM
- R54 pad 1: ~ -> +3.3V
- R54 pad 2: Net-(C47-Pad1) -> Net-(C49-Pad1)
- R58 pad 1: ~ -> +3.3V
- R59 pad 1: ~ -> +3.3V
- T14 pad 2: ~ -> +3.3V
- TP23 pad 1: ~ -> +3.3VSTM
- TP24 pad 1: ~ -> +3.3V
- U10 pad 5: ~ -> +3.3VSTM
- U11 pad 1: ~ -> +3.3VSTM
- U11 pad 13: ~ -> +3.3VSTM
- U11 pad 19: ~ -> +3.3VSTM
- U11 pad 32: ~ -> +3.3VSTM
- U11 pad 48: ~ -> +3.3VSTM
- U11 pad 64: ~ -> +3.3VSTM
- U13 pad 4: ~ -> +3.3VSTM
- U14 pad 4: ~ -> +3.3V
- U17 pad 7: Net-(R51-Pad1) -> Net-(C44-Pad1)
- U18 pad 8: ~ -> +3.3VSTM
- U19 pad 1: Net-(C47-Pad1) -> Net-(C49-Pad1)
- U19 pad 8: ~ -> +3.3V
- U7 pad 20: ~ -> +3.3V
- U8 pad 20: ~ -> +3.3V
- U9 pad 8: ~ -> +3.3V
Routing:
- net +3.3V: track 0.00 -> 292.3 mm, vias 0 -> 15
- net VBAT: track 101.8 -> 393.9 mm, vias 2 -> 20
- net GND: track 759.1 -> 1020.0 mm, vias 16 -> 23
- net +3.3VSTM: track 0.00 -> 157.5 mm, vias 0 -> 11
- net /URT1_TX: track 0.00 -> 129.9 mm, vias 0 -> 2
- net /485A: track 2.33 -> 131.0 mm, vias 0 -> 7
- net /SPI_MISO: track 0.00 -> 127.6 mm, vias 0 -> 7
- net /GSM_DTR: track 0.00 -> 124.9 mm, vias 0 -> 3
- net /485B: track 2.33 -> 127.1 mm, vias 0 -> 7
- net ~: track 316.9 -> 193.4 mm, vias 11 -> 6
- net Net-(R52-Pad1): track 0.00 -> 119.2 mm, vias 0 -> 3
- net /SPI_MOSI: track 0.00 -> 118.5 mm, vias 0 -> 5
- net /SPI_CLK: track 0.00 -> 115.6 mm, vias 0 -> 3
- net /CS_ESP: track 0.00 -> 79.1 mm, vias 0 -> 3
- net Net-(R57-Pad2): track 0.00 -> 78.6 mm, vias 0 -> 1
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- added copper zone on F.Cu, net GND
- added copper zone on F.Cu, net VBAT
Other:
- board size 150 x 100 mm -> 111 x 100 mm
- net class 120 mils added: clearance 0.508, trace_width 3.048, via_dia 3, via_drill 1.5
- net class 20 mils added: clearance 0.254, trace_width 0.508, via_dia 0.6, via_drill 0.3
- net class 50 mils added: clearance 0.254, trace_width 1.27, via_dia 1.4, via_drill 0.7
- net class Default: clearance 0.2 -> 0.127; trace_width 0.25 -> 0.2032
- net class gruba removed
- rule trace_clearance: 0.2 -> 0.127

Commit message: sprawdzanie drc pcb
Parts:
- removed TP19, TP20: TEST, Measurement_Points:Measurement_Point_Round-SMD-Pad_Big
- moved TP27 106.0 mm to (75.7, 90.4)
- moved TP28 102.3 mm to (17.8, 102.9)
- moved TP21 99.3 mm to (75.7, 96.0)
- moved TP16 95.0 mm to (37.3, 127.5)
- moved TP25 92.3 mm to (101.9, 98.0)
- moved TP22 88.1 mm to (116.1, 114.0)
- moved TP30 86.5 mm to (20.1, 157.5)
- moved TP24 85.2 mm to (75.9, 108.5)
- moved TP31 85.1 mm to (20.1, 152.9)
- moved TP26 81.1 mm to (99.3, 101.3)
- moved TP23 80.4 mm to (49.8, 103.9)
- moved TP18 73.7 mm to (80.0, 119.4)
- moved TP8 71.8 mm to (54.1, 139.2)
- moved TP7 71.7 mm to (50.3, 139.2)
- moved TP11 69.5 mm to (54.1, 144.5)
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Routing:
- net Net-(R57-Pad1): track 21.0 -> 83.7 mm, vias 2 -> 3
- net GND: track 1020.0 -> 1064.8 mm
- net /VBON4: track 27.5 -> 66.2 mm, vias 0 -> 4
- net /VBON5: track 34.6 -> 70.4 mm, vias 0 -> 4
- net /VBON6: track 52.8 -> 83.9 mm, vias 0 -> 4
- net /VBON3: track 22.9 -> 47.5 mm, vias 0 -> 2
- net /485A: track 131.0 -> 154.4 mm, vias 7 -> 9
- net /485B: track 127.1 -> 146.9 mm, vias 7 -> 9
- net /DHT22_DATA: track 2.58 -> 22.0 mm
- net Net-(R57-Pad2): track 78.6 -> 60.7 mm
- net /RESET: track 20.0 -> 36.5 mm, vias 2 -> 4
- net /URT1_RX: track 2.46 -> 16.5 mm, vias 0 -> 2
- net /URT1_TX: track 129.9 -> 141.3 mm, vias 2 -> 3
- net /VBON2: track 34.9 -> 46.2 mm, vias 0 -> 2
- net +3.3V: track 292.3 -> 303.6 mm, vias 15 -> 17
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- removed copper zone on F.Cu, net VBAT
Other:
- net class 120 mils: clearance 0.508 -> 0.127
- net class 20 mils: clearance 0.254 -> 0.127
- rule trace_min: 0.2 -> 0.127
- rule via_min_size: 0.4 -> 0.2

Commit message: +creo, po naprawie w pracy
Parts:
- added REF**: MountingHole_2.7mm_M2.5, Mounting_Holes:MountingHole_2.7mm_M2.5, F.Cu at (119.0, 131.5)
- added REF**: MountingHole_2.7mm_M2.5, Mounting_Holes:MountingHole_2.7mm_M2.5, F.Cu at (21.0, 159.5)
- added REF**: MountingHole_2.7mm_M2.5, Mounting_Holes:MountingHole_2.7mm_M2.5, F.Cu at (120.0, 79.0)
- added REF**: MountingHole_2.7mm_M2.5, Mounting_Holes:MountingHole_2.7mm_M2.5, F.Cu at (20.0, 79.0)
- moved J8 75.8 mm to (49.1, 131.4), turned to 270 degrees
- moved R36 54.7 mm to (60.2, 129.3), turned to 180 degrees
- moved R57 22.6 mm to (112.3, 76.3), turned to 0 degrees
- moved U20 18.3 mm to (110.5, 91.6), turned to 270 degrees
- moved TP23 12.1 mm to (58.8, 95.8)
- moved R31 6.70 mm to (113.7, 135.8), turned to 270 degrees
- moved TP13 4.60 mm to (18.8, 170.2)
- moved TP14 4.60 mm to (22.9, 170.2)
- moved TP22 3.99 mm to (119.8, 112.5)
- moved F3 3.81 mm to (61.0, 161.3)
- moved T3 3.81 mm to (61.0, 157.5)
- moved T9 3.81 mm to (61.0, 150.1)
- moved C1 3.81 mm to (37.4, 150.9)
- moved C10 3.81 mm to (81.3, 150.9)
- moved C11 3.81 mm to (97.0, 150.9)
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Routing:
- net Net-(R57-Pad2): track 60.7 -> 99.8 mm
- net Net-(D3-Pad1): track 33.5 -> 57.0 mm
- net GND: track 1064.8 -> 1085.5 mm, vias 23 -> 21
- net Net-(U17-Pad12): track 59.8 -> 77.2 mm
- net Net-(U17-Pad13): track 69.9 -> 82.6 mm
- net +3.3VSTM: track 167.6 -> 178.4 mm, vias 13 -> 14
- net Net-(D2-Pad1): track 47.9 -> 41.3 mm
- net Net-(J7-Pad1): track 2.34 -> 8.40 mm
- net /VBON6: track 83.9 -> 79.1 mm
- net Net-(R57-Pad1): track 83.7 -> 88.1 mm
- net Net-(P3-Pad1): track 33.6 -> 29.2 mm
- net /RTC_BAT: track 11.5 -> 7.10 mm
- net /ESP_ON: track 77.4 -> 81.3 mm
- net /33ON2: track 24.1 -> 27.9 mm
- net Net-(P3-Pad3): track 34.3 -> 30.6 mm
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Other:
- board size 111 x 100 mm -> 110 x 100 mm
- rule trace_min: 0.127 -> 0.2032
