File: test.kicad_pcb (KiCad board)
At the start: 2 copper layers, 110 x 100 mm, 213 parts, among them J1 HSP2_MX-502584-0670, J10 Gniazdo programatora SWD, J11 Gniazdo akumulatora, J12 Gniazdo akumulatora, J13 SIMHOLDER, J14 BTN1, J15 BTN2, J2 HSP2_MX-502584-0670, J3 HSP2_MX-502584-0670, J4 HSP2_MX-502584-0670, J5 HSP2_MX-502584-0670, J6 HSP2_MX-502584-0670, J7 CONN_02X01, J8 CONN_02X01, J9 microSD, T1 IRLML6401, T10 BSS138, T11 BSS138, T12 BSS138, T13 BSS138, T14 FDV304P, T2 IRLML6401, T3 IRLML6401, T4 IRLML6401, T5 IRLML6401, T6 IRLML6401, T7 BSS138, T8 BSS138, T9 BSS138, U1 MCP1755T-3302E/DC, U10 TPS3823, U11 STM32L051R8, U12 DS3231SN, U13 MCP1755T-3302E/DC, U14 MCP1755T-3302E/DC, U15 MIC29302, U16 DHT22, U17 M590E, U18 S25FL1275ABMGI101, U19 ESP-WROOM-32, U2 MCP1755T-3302E/DC, U3 MCP1755T-3302E/DC, U4 MCP1755T-3302E/DC, U5 MCP1755T-3302E/DC, U6 MCP1755T-3302E/DC, U7 74LVX373M, U8 74LVX373M, U9 MAX3485, Y1 32.768 kHz, Y2 8 MHz

Commit message: routowanie esp32
Parts:
- moved R37 63.0 mm to (127.6, 116.6)
- moved TP2 22.1 mm to (149.7, 68.6)
- moved TP1 21.7 mm to (153.0, 66.2)
- moved TP29 21.0 mm to (156.8, 67.5)
- moved C50 4.53 mm to (156.5, 62.1), turned to 270 degrees
- moved C52 4.51 mm to (158.0, 62.1), turned to 270 degrees
- moved R54 3.05 mm to (161.1, 73.3)
- moved R58 2.92 mm to (161.3, 75.3), turned to 180 degrees
- moved R61 1.82 mm to (152.5, 74.0)
- moved R62 1.45 mm to (154.1, 74.0)
- moved R59 0.38 mm to (155.8, 74.0)
Routing:
- net /URT2_RX: track 15.9 -> 58.5 mm, vias 3 -> 7
- net /URT2_TX: track 13.9 -> 51.0 mm, vias 3 -> 6
- net /ESP_IO0: track 14.2 -> 47.9 mm, vias 0 -> 4
- net /GSM_STAB_EN: track 94.3 -> 60.7 mm, vias 2 -> 4
- net /ESP_IO2: track 12.5 -> 45.5 mm, vias 0 -> 4
- net GND: track 1069.6 -> 1098.2 mm, vias 25 -> 24
- net +3.3V: track 280.0 -> 257.2 mm
- net Net-(J13-Pad3): track 74.9 -> 92.9 mm
- net Net-(J13-Pad2): track 79.1 -> 96.1 mm
- net Net-(J13-Pad6): track 82.8 -> 97.9 mm, vias 2 -> 3
- net /CS_ESP: track 59.2 -> 74.0 mm
- net /SPI_CLK: track 94.3 -> 81.7 mm
- net Net-(R51-Pad1): track 113.9 -> 102.6 mm
- net /URT1_TX: track 137.1 -> 126.0 mm
- net Net-(R52-Pad1): track 118.0 -> 107.0 mm
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