File: test.kicad_pcb (KiCad board)
At the start: 2 copper layers, 110 x 100 mm, 213 parts, among them J1 HSP2_MX-502584-0670, J10 Gniazdo programatora SWD, J11 Gniazdo akumulatora, J12 Gniazdo akumulatora, J13 SIMHOLDER, J14 BTN1, J15 BTN2, J2 HSP2_MX-502584-0670, J3 HSP2_MX-502584-0670, J4 HSP2_MX-502584-0670, J5 HSP2_MX-502584-0670, J6 HSP2_MX-502584-0670, J7 CONN_02X01, J8 CONN_02X01, J9 microSD, T1 IRLML6401, T10 BSS138, T11 BSS138, T12 BSS138, T13 BSS138, T14 FDV304P, T2 IRLML6401, T3 IRLML6401, T4 IRLML6401, T5 IRLML6401, T6 IRLML6401, T7 BSS138, T8 BSS138, T9 BSS138, U1 MCP1755T-3302E/DC, U10 TPS3823, U11 STM32L051R8, U12 DS3231SN, U13 MCP1755T-3302E/DC, U14 MCP1755T-3302E/DC, U15 MIC29302, U16 DHT22, U17 M590E, U18 S25FL1275ABMGI101, U19 ESP-WROOM-32, U2 MCP1755T-3302E/DC, U3 MCP1755T-3302E/DC, U4 MCP1755T-3302E/DC, U5 MCP1755T-3302E/DC, U6 MCP1755T-3302E/DC, U7 74LVX373M, U8 74LVX373M, U9 MAX3485, Y1 32.768 kHz, Y2 8 MHz

Commit message: esp32 i btn zrutowanie calkowicie
Parts:
- added TP23: TEST, Measurement_Points:Measurement_Point_Round-SMD-Pad_Big, F.Cu at (187.0, 80.5)
- added TP3: TEST, Measurement_Points:Measurement_Point_Round-SMD-Pad_Big, F.Cu at (168.8, 73.6)
- added TP4: TEST, Measurement_Points:Measurement_Point_Round-SMD-Pad_Big, F.Cu at (166.7, 76.9)
- added TP5: TEST, Measurement_Points:Measurement_Point_Round-SMD-Pad_Big, F.Cu at (161.2, 67.2)
- moved C54 1.41 mm to (190.7, 98.8)
- moved U18 1.27 mm to (194.0, 99.0)
- moved J15 0.82 mm to (148.4, 103.4)
Routing:
- net /GSM_STAB_EN: track 60.7 -> 126.2 mm, vias 4 -> 2
- net /BTN2: track 0.00 -> 50.2 mm, vias 0 -> 2
- net GND: track 1098.2 -> 1125.5 mm
- net /BTN1: track 1.98 -> 26.9 mm, vias 0 -> 2
- net +3.3V: track 257.2 -> 275.0 mm
- net /SPI_CLK: track 81.7 -> 91.1 mm
- net /SPI_MOSI: track 90.7 -> 99.8 mm, vias 4 -> 6
- net /SPI_MISO: track 98.3 -> 107.0 mm
- net /VON3: track 66.1 -> 61.1 mm
- net Net-(C31-Pad1): track 15.7 -> 20.6 mm
- net /VON2: track 66.0 -> 61.4 mm
- net /33LOE: track 53.1 -> 48.8 mm
- net /VON1: track 66.8 -> 62.9 mm
- net Net-(D3-Pad1): track 58.7 -> 56.0 mm
- net +3.3VSTM: track 172.5 -> 174.6 mm
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Other:
- rule trace_min: 0.2032 -> 0.508

Commit message: wersja final, freeze wyslana do technoservice
Parts:
- removed the ? at (109.0, 141.0)
- added ?: myfid1, footprints:myfid1, F.Cu at (105.0, 142.0)
- added ?: myfid1, footprints:myfid1, F.Cu at (203.0, 62.0)
- moved C31 14.2 mm to (153.3, 92.9)
- moved C37 11.4 mm to (153.4, 91.1)
- moved C32 11.0 mm to (140.4, 90.7)
- moved C36 10.9 mm to (143.3, 90.7)
- moved J12 5.94 mm to (106.6, 108.5)
- moved J11 5.84 mm to (106.7, 89.5)
- moved J7 4.26 mm to (206.4, 122.3)
- moved J8 4.26 mm to (134.4, 103.1)
- moved J14 4.26 mm to (181.7, 104.3)
- moved J15 4.26 mm to (148.7, 99.2)
Routing:
- net Net-(C32-Pad1): track 25.3 -> 9.83 mm
- net Net-(C31-Pad1): track 20.6 -> 7.26 mm
- net GND: track 1125.5 -> 1112.9 mm, vias 24 -> 23
- net Net-(C45-Pad1): track 127.3 -> 125.8 mm
- net +3.3VSTM: track 174.6 -> 173.6 mm, vias 12 -> 14
Other:
- net class Default: via_drill 0.2 -> 0.15
- rule trace_min: 0.508 -> 0.2032
- rule via_min_drill: 0.2 -> 0.15
- rule via_min_size: 0.2 -> 0.4
- board text added: "HSP2 rev. 1.0"
- board text added: "PEO_1736"

Commit message: zmiana flash
Parts:
- U18: value S25FL1275ABMGI101 -> AT45DB161E-SSHD-T; footprint footprints:SO-8 -> footprints:8-lead_JEDEC_SOIC
- turned U18 to 90 degrees
Connections:
- U11 pad 58: Net-(U11-Pad58) -> FLASH_RESET
- U18 pad 1: /CS_FLA -> /SPI_CLK
- U18 pad 2: /SPI_MISO -> /SPI_MOSI
- U18 pad 3: Net-(U18-Pad3) -> FLASH_RESET
- U18 pad 4: GND -> /CS_FLA
- U18 pad 5: /SPI_MOSI -> Net-(U18-Pad5)
- U18 pad 6: /SPI_CLK -> +3.3VSTM
- U18 pad 7: Net-(U18-Pad7) -> GND
- U18 pad 8: +3.3VSTM -> /SPI_MISO
Routing:
- net FLASH_RESET: track 0.00 -> 35.0 mm, vias 0 -> 6
- net /SPI_CLK: track 91.1 -> 77.6 mm
- net /SPI_MOSI: track 99.8 -> 86.6 mm, vias 6 -> 4
- net /CS_FLA: track 31.7 -> 24.2 mm
- net /SPI_MISO: track 107.0 -> 110.0 mm
- net +3.3VSTM: track 173.6 -> 176.4 mm, vias 14 -> 16
- net GND: track 1112.9 -> 1114.5 mm
Other:
- rule pad_to_mask_clearance: 0.2 -> 0.1

Commit message: poprawione przelotki i ścieżki
Parts:
- moved C21 1.70 mm to (167.9, 88.9)
- moved J8 1.16 mm to (135.5, 103.2)
Connections:
- U18 pad 1: /SPI_CLK -> /SPI_MOSI
- U18 pad 2: /SPI_MOSI -> /SPI_CLK
Routing:
- net /SPI_CLK: track 77.6 -> 90.7 mm, vias 2 -> 4
- net /SPI_MOSI: track 86.6 -> 98.8 mm, vias 4 -> 6
- net Net-(C32-Pad1): track 9.83 -> 12.7 mm
- net GND: track 1114.5 -> 1112.0 mm
- net +3.3V: track 274.6 -> 273.1 mm
- net Net-(D3-Pad1): track 56.1 -> 55.0 mm
- net Net-(C14-Pad1): track 11.6 -> 12.2 mm
- net /I2C2_SDA: track 39.2 -> 38.6 mm
Other:
- board text added: "HSP2 rev. 1.1"
- board text removed: "HSP2 rev. 1.0"
